File: watch/pcb/non_chargeable/non_chargeable.kicad_pcb (KiCad board)
At the start: 2 copper layers, 39.9 x 41.8 mm, 11 parts, among them U2 ATTINY85-20SUR

Commit message: non- chargeable
Parts:
- removed BT1: BT1, Battery:BatteryHolder_Keystone_1060_1x2032
- removed RST1: RST, Button_Switch_SMD:SW_Tactile_SPST_NO_Straight_CK_PTS636Sx25SMTRLFS
- removed SEL1: SEL, Button_Switch_SMD:SW_Tactile_SPST_NO_Straight_CK_PTS636Sx25SMTRLFS
- removed SET1: SET, Button_Switch_SMD:SW_Tactile_SPST_NO_Straight_CK_PTS636Sx25SMTRLFS
- removed WK1: WK, Button_Switch_SMD:SW_Tactile_SPST_NO_Straight_CK_PTS636Sx25SMTRLFS
- added BT2: 1059, BatteryHolder_Keystone_1059_THT:BatteryHolder_Keystone_1059_THT, B.Cu at (152.5, 91.7)
- added RST: RST, My_Tactile_Switch:PTS636_SM43_LFS, F.Cu at (147.1, 68.1)
- added SEL: SEL, My_Tactile_Switch:PTS636_SM43_LFS, F.Cu at (142.3, 68.1)
- added SET: SET, My_Tactile_Switch:PTS636_SM43_LFS, F.Cu at (137.4, 68.1)
- added WK: WK, My_Tactile_Switch:PTS636_SM43_LFS, F.Cu at (132.6, 68.1)
- U2: footprint My_ATTINY:8S2_ATM-L -> Package_DIP:DIP-8_W7.62mm_Socket
- moved U2 6.25 mm to (151.1, 75.0), turned to 90 degrees
Connections:
- net MOSI renamed SDA
- U2 pad 6: MISO -> WAKE
Routing:
- net SCK: track 0.00 -> 37.2 mm
- net SDA: track 0.00 -> 36.7 mm
- net WAKE: track 0.00 -> 26.3 mm
- net SET: track 0.00 -> 22.0 mm
- net SELECT: track 0.00 -> 13.5 mm
- net RESET: track 0.00 -> 4.14 mm
Other:
- board text added: "https://tinyurl.com/22p6cwfd"
- board text removed: "Parten Ranch Robotics"
