File: watch/pcb/non_chargeable/non_chargeable.kicad_sch (KiCad schematic)
At the start: 12 parts, among them J2 PROG, U2 ATTINY85-20SUR

Commit message: non- chargeable
Parts:
- removed BT1: BT1, Battery:BatteryHolder_Keystone_1060_1x2032, symbol Device:Battery_Cell
- removed J2: PROG, JST_PH_1x06_2mm_horizontal:JST_PH_1x06_2mm_horizontal.pretty, symbol JST_PH_1x06_2mm_horizontal:S6B-PH-SM4-TB_LF__SN_
- added BT2: 1059, BatteryHolder_Keystone_1059_THT:BatteryHolder_Keystone_1059_THT, symbol BatteryHolder_Keystone_1059:1059
- H1, H2, H3, H4, OLED_DISPLAY1: now fitted; now in the parts list
- RST1, SEL1, SET1, WK1: footprint Button_Switch_SMD:SW_Tactile_SPST_NO_Straight_CK_PTS636Sx25SMTRLFS -> My_Tactile_Switch:PTS636_SM43_LFS
- U2: footprint My_ATTINY:8S2_ATM-L -> Package_DIP:DIP-8_W7.62mm_Socket
Connections:
- net GND: now also BT2.N
- net VCC: now also BT2.P1
- net MISO renamed WAKE
- net MOSI renamed SDA
Other:
- note removed: "Programming"
- moved on the sheet: RST1, SEL1, SET1, U2, WK1
